Commit message: Adapted for simulation

File: yumi_description/urdf/Grippers/yumi_servo_gripper.xacro (robot description, xacro)
@@ -11,4 +11,5 @@
     <xacro:property name="max_gripper_effort" value="20"/>
     <xacro:property name="max_gripper_velocity" value="2"/>
+    <xacro:property name="M_PI" value="3.1415926535897931" />
   <xacro:macro name="yumi_servo_gripper" params="parent name hardware_interface *origin">
     <!--joint between {parent} and base-->
@@ -27,5 +28,10 @@
         <origin xyz="0 0 0" rpy="0 0 0"/>
         <geometry>
-          <mesh filename="package://yumi_description/meshes/gripper/base.stl"/>
+          <xacro:if value="${(name == 'gripper_l')}">
+            <mesh filename="package://yumi_description/meshes/gripper/base_with_case_l.stl"/>
+          </xacro:if>
+          <xacro:if value="${(name == 'gripper_r')}">
+            <mesh filename="package://yumi_description/meshes/gripper/base_with_case_r.stl"/>
+          </xacro:if>
         </geometry>
         <material name="Light_Grey"/>
@@ -34,5 +40,10 @@
         <origin xyz="0 0 0" rpy="0 0 0"/>
         <geometry>
-          <mesh filename="package://yumi_description/meshes/gripper/coarse/base.stl"/>
+          <xacro:if value="${(name == 'gripper_l')}">
+            <mesh filename="package://yumi_description/meshes/gripper/coarse/base_with_case_l.stl"/>
+          </xacro:if>
+          <xacro:if value="${(name == 'gripper_r')}">
+            <mesh filename="package://yumi_description/meshes/gripper/coarse/base_with_case_r.stl"/>
+          </xacro:if>
         </geometry>
         <material name="Light_Grey"/>
@@ -54,5 +65,6 @@
         <origin xyz="0 0 0" rpy="0 0 0"/>
         <geometry>
-          <mesh filename="package://yumi_description/meshes/gripper/finger.stl"/>
+          <mesh filename="package://yumi_description/meshes/gripper/finger_long.stl"/>
+          <!-- <mesh filename="package://yumi_description/meshes/gripper/finger.stl"/> -->
         </geometry>
         <material name="Blue"/>
@@ -61,5 +73,6 @@
         <origin xyz="0 0 0" rpy="0 0 0"/>
         <geometry>
-          <mesh filename="package://yumi_description/meshes/gripper/coarse/finger.stl"/>
+          <mesh filename="package://yumi_description/meshes/gripper/coarse/finger_long.stl"/>
+          <!-- <mesh filename="package://yumi_description/meshes/gripper/coarse/finger.stl"/> -->
         </geometry>
         <material name="Blue"/>
@@ -82,5 +95,6 @@
         <origin xyz="0 0 0" rpy="0 0 0"/>
         <geometry>
-          <mesh filename="package://yumi_description/meshes/gripper/finger.stl"/>
+          <mesh filename="package://yumi_description/meshes/gripper/finger_long.stl"/>
+          <!-- <mesh filename="package://yumi_description/meshes/gripper/finger.stl"/> -->
         </geometry>
         <material name="Blue"/>
@@ -89,7 +103,39 @@
         <origin xyz="0 0 0" rpy="0 0 0"/>
         <geometry>
-          <mesh filename="package://yumi_description/meshes/gripper/coarse/finger.stl"/>
+          <mesh filename="package://yumi_description/meshes/gripper/coarse/finger_long.stl"/>
+          <!-- <mesh filename="package://yumi_description/meshes/gripper/coarse/finger.stl"/> -->
         </geometry>
         <material name="Blue"/>
+      </collision>
+    </link>
+    <!-- joint between body and camera -->
+    <joint name="${name}_camera_joint" type="fixed">
+      <parent link="${name}_base"/>
+      <child link="${name}_camera_link"/>
+      <xacro:if value="${(name == 'gripper_l')}">
+        <origin xyz="0.0171 0.0533 0.0535" rpy="1.1805 -1.5625 -2.7600"/>
+      </xacro:if>
+      <xacro:if value="${(name == 'gripper_r')}">
+        <origin xyz="-0.0115 -0.0544 0.0603" rpy="-0.3901 -1.5426 1.9291"/>
+      </xacro:if>
+    </joint>
+    <link name="${name}_camera_link">
+      <inertial>
+        <origin xyz="0 0 0" rpy="0 0 0"/>
+        <mass value="1"/>
+        <inertia ixx="0.1"  ixy="0"  ixz="0" iyy="0.1" iyz="0" izz="0.1" />
+      </inertial>
+      <visual>
+        <origin xyz="4.3e-3 -0.0175 0" rpy="${M_PI/2} 0 ${M_PI/2}"/>
+        <geometry>
+          <mesh filename="package://yumi_description/meshes/d435.dae" scale="1 1 1"/>
+        </geometry>
+        <material name="Grey"/>
+      </visual>
+      <collision>
+        <origin xyz="0 -0.0175 0" rpy="0 0 0"/>
+        <geometry>
+          <box size="0.02505 0.090 0.025"/>
+        </geometry>
       </collision>
     </link>

File: yumi_description/urdf/yumi.urdf.xacro (robot description, xacro)
@@ -11,7 +11,16 @@
   <!-- Import Gazebo plugins -->
   <xacro:include filename="$(find yumi_description)/urdf/Gazebo/gazebo.urdf.xacro"/>
+  <xacro:property name="yumi_setup" value="$(arg yumi_setup)" />
+  <xacro:if value="${yumi_setup == 'default'}">
+    <xacro:property name="yumi_parent" value="world" />
+    <link name="world"/>
+    <joint name="world_joint" type="fixed">
+      <parent link="world"/>
+      <child link="yumi_base_link"/>
+      <origin xyz="0 0 0" rpy="0 0 0" />
+    </joint>
+  </xacro:if>
   <!--yumi-->
   <xacro:yumi name="yumi" hardware_interface="hardware_interface/$(arg arms_interface)" parent="${yumi_parent}" >
-    <origin xyz="0 0 0.1" rpy="0 0 0" />
   </xacro:yumi>
   <!--right gripper-->
@@ -23,16 +32,6 @@
     <origin xyz="0 0 0.007" rpy="0 0 ${PI}" />
   </xacro:yumi_servo_gripper>
-  <xacro:property name="yumi_setup" value="$(arg yumi_setup)" />
   <xacro:if value="${yumi_setup == 'robot_centric'}">
   	<!-- Pure YuMi URDF, with no joints connecting it to any other robot or pedestal. Neither accessories. -->
   </xacro:if>
-  <xacro:if value="${yumi_setup == 'default'}">
-    <xacro:property name="yumi_parent" value="world" />
-    <link name="world"/>
-    <joint name="world_joint" type="fixed">
-      <parent link="world"/>
-      <child link="yumi_base_link"/>
-      <origin xyz="0 0 0.1" rpy="0 0 0" />
-    </joint>
-  </xacro:if>
 </robot>

File: yumi_description/urdf/yumi.xacro (robot description, xacro)
@@ -8,5 +8,5 @@
   <xacro:property name="joint_damping" value="0.5" />
   <xacro:property name="max_effort" value="300"/>
-  <xacro:macro name="yumi" params="parent name hardware_interface *origin">
+  <xacro:macro name="yumi" params="parent name hardware_interface">
     <link name="yumi_base_link"></link>
     <joint name="${name}_base_link_to_body" type="fixed">
@@ -472,4 +472,30 @@
       </collision>
     </link>
+    <!-- joint between body and camera -->
+    <joint name="${name}_camera_joint" type="fixed">
+      <parent link="${name}_base_link"/>
+      <child link="${name}_camera_link"/>
+      <origin xyz="0.1015 -0.0030 0.3332" rpy="-0.0081 0.6795 0.0112"/>
+    </joint>
+    <link name="${name}_camera_link">
+      <inertial>
+        <origin xyz="0 0 0" rpy="0 0 0"/>
+        <mass value="1"/>
+        <inertia ixx="0.1"  ixy="0"  ixz="0" iyy="0.1" iyz="0" izz="0.1" />
+      </inertial>
+      <visual>
+        <origin xyz="0.0045 0 0.0099" rpy="${M_PI/2} 0 ${M_PI/2}"/>
+        <geometry>
+          <mesh filename="package://yumi_description/meshes/l515.dae" />
+        </geometry>
+        <material name="Grey"/>
+      </visual>
+      <collision>
+        <origin xyz="-0.9935 0 0.0099" rpy="${M_PI/2} 0 ${M_PI/2}"/>
+        <geometry>
+          <cylinder radius="0.0305" length="0.026"/>
+        </geometry>
+      </collision>
+    </link>
     <!--Extensions -->
     <xacro:yumi_gazebo name="${name}" />
